File: kicad/pga2350-breakout.kicad_sch (KiCad schematic)
At the start: 6 parts, among them J1 Conn_01x02_Pin, J2 Conn_02x05_Odd_Even, J3 Conn_01x02_Pin, J4 Conn_01x05_Pin, J5 Conn_02x24_Counter_Clockwise

Commit message: initial routing, DRC all clear
Parts:
- removed J5: Conn_02x24_Counter_Clockwise, symbol Connector_Generic:Conn_02x24_Counter_Clockwise
- added J10, J5, J6, J7, J8: Conn_02x05_Counter_Clockwise, Connector_PinSocket_2.54mm:PinSocket_2x05_P2.54mm_Vertical, symbol Connector_Generic:Conn_02x05_Counter_Clockwise
Connections:
- net GND: now also J2.3 (Pin_3), J2.4 (Pin_4), J2.7 (Pin_7), J2.8 (Pin_8), J8.10 (Pin_10)
- net GP0: now also J10.1 (Pin_1); no longer U1.62 (GP1)
- net GP10: now reaches U1.10 (GP10)
- net GP10: now also J5.1 (Pin_1)
- net GP11: now reaches U1.11 (GP11)
- net GP11: now also J5.2 (Pin_2)
- net GP12: now reaches U1.12 (GP12)
- net GP12: now also J5.3 (Pin_3)
- net GP13: now reaches U1.13 (GP13)
- net GP13: now also J5.4 (Pin_4)
- net GP14: now reaches U1.14 (GP14)
- net GP14: now also J5.5 (Pin_5)
- net GP15: now reaches U1.15 (GP15)
- net GP15: now also J5.6 (Pin_6)
- net GP16: now reaches U1.16 (GP16)
- net GP16: now also J5.7 (Pin_7)
- net GP17: now reaches U1.17 (GP17)
- net GP17: now also J5.8 (Pin_8)
- net GP18: now reaches U1.19 (GP18)
- net GP18: now also J5.9 (Pin_9)
- net GP2: now reaches U1.2 (GP2)
- net GP2: now also J10.3 (Pin_3)
- net GP19: now reaches U1.20 (GP19)
- net GP19: now also J5.10 (Pin_10)
- net GP20: now reaches U1.21 (GP20)
- net GP20: now also J6.1 (Pin_1)
- net GP21: now reaches U1.22 (GP21)
- net GP21: now also J6.2 (Pin_2)
- net GP22: now reaches U1.23 (GP22)
- net GP22: now also J6.3 (Pin_3)
- net GP23: now reaches U1.24 (GP23)
- net GP23: now also J6.4 (Pin_4)
- net GP24: now reaches U1.25 (GP24)
- net GP24: now also J6.5 (Pin_5)
- net GP25: now reaches U1.26 (GP25)
- net GP25: now also J6.6 (Pin_6)
- net GP26: now reaches U1.27 (GP26)
- net GP26: now also J6.7 (Pin_7)
- net GP27: now reaches U1.28 (GP27)
- net GP27: now also J6.8 (Pin_8)
- net GP28: now reaches U1.29 (GP28)
- net GP28: now also J6.9 (Pin_9)
- net GP3: now reaches U1.3 (GP3)
- net GP3: now also J10.4 (Pin_4)
- net GP29: now reaches U1.30 (GP29)
- net GP29: now also J6.10 (Pin_10)
- net GP30: now reaches U1.31 (GP30)
- net GP30: now also J7.1 (Pin_1)
- net GP31: now reaches U1.32 (GP31)
- net GP31: now also J7.2 (Pin_2)
- net GP32: now reaches U1.34 (GP32)
- net GP32: now also J7.3 (Pin_3)
- net GP33: now reaches U1.35 (GP33)
- net GP33: now also J7.4 (Pin_4)
- net GP34: now reaches U1.36 (GP34)
- net GP34: now also J7.5 (Pin_5)
- net GP35: now reaches U1.37 (GP35)
- net GP35: now also J7.6 (Pin_6)
- net GP36: now reaches U1.38 (GP36)
- net GP36: now also J7.7 (Pin_7)
- net GP37: now reaches U1.39 (GP37)
- net GP37: now also J7.8 (Pin_8)
- net GP4: now reaches U1.4 (GP4)
- net GP4: now also J10.5 (Pin_5)
- net GP38: now reaches U1.40 (GP38)
- net GP38: now also J7.9 (Pin_9)
- net GP39: now reaches U1.41 (GP39)
- net GP39: now also J7.10 (Pin_10)
- net GP40: now reaches U1.42 (GP40)
- net GP40: now also J8.1 (Pin_1)
- net GP41: now reaches U1.43 (GP41)
- net GP41: now also J8.2 (Pin_2)
- net GP42: now reaches U1.44 (GP42)
- net GP42: now also J8.3 (Pin_3)
- net GP43: now reaches U1.45 (GP43)
- net GP43: now also J8.4 (Pin_4)
- net GP44: now reaches U1.46 (GP44)
- net GP44: now also J8.5 (Pin_5)
- net GP45: now reaches U1.47 (GP45)
- net GP45: now also J8.6 (Pin_6)
- net GP46: now reaches U1.49 (GP46)
- net GP46: now also J8.7 (Pin_7)
- net GP5: now reaches U1.5 (GP5)
- net GP5: now also J10.6 (Pin_6)
- net GP47: now reaches U1.50 (GP47)
- net GP47: now also J8.8 (Pin_8)
- net BOOTSETL: now reaches U1.51 (BOOTSEL)
- net SWDIO: now reaches U1.52 (SWDIO)
- net SWCLK: now reaches U1.55 (SWCLK)
- net RUN: now reaches U1.56 (RUN)
- net ADC_VREF: now reaches U1.57 (ADC_VREF)
- net ADC_VREF: now also J8.9 (Pin_9)
- net 3V3_EN: now reaches U1.58 (3V3_EN)
- net GP6: now reaches U1.6 (GP6)
- net GP6: now also J10.7 (Pin_7)
- net GP7: now reaches U1.7 (GP7)
- net GP7: now also J10.8 (Pin_8)
- net GP8: now reaches U1.8 (GP8)
- net GP8: now also J10.9 (Pin_9)
- net GP9: now reaches U1.9 (GP9)
- net GP9: now also J10.10 (Pin_10)
- new net GP1: J10.2 (Pin_2), U1.62 (GP1)
Other:
- moved on the sheet: J1, J3

Commit message: save production version 1.0
Parts:
- added J11, J9: Conn_01x02_Pin, allen-synthesis:pin-socket-2.54mm-01x02, symbol Connector:Conn_01x02_Pin
- added J12: Conn_01x03_Pin, allen-synthesis:pin-header-2.54mm-01x03, symbol Connector:Conn_01x03_Pin
- J1, J3: footprint Connector_PinSocket_2.54mm:PinSocket_1x02_P2.54mm_Vertical -> allen-synthesis:pin-socket-2.54mm-01x02
- J10, J5, J6, J7, J8: footprint Connector_PinSocket_2.54mm:PinSocket_2x05_P2.54mm_Vertical -> allen-synthesis:pin-socket-2.54mm-02x05
- J4: footprint Connector_PinHeader_2.54mm:PinHeader_1x05_P2.54mm_Vertical -> allen-synthesis:pin-header-2.54mm-01x05
Connections:
- net BOOTSETL: now also J9.1 (Pin_1)
- net GND: now also J11.2 (Pin_2), J12.2 (Pin_2), J9.2 (Pin_2)
- net RUN: now also J11.1 (Pin_1)
- net SWCLK: now also J12.3 (Pin_3)
- net SWDIO: now also J12.1 (Pin_1)
Other:
- moved on the sheet: J1, J10, J2, J3, J5, J6, J7, J8
